File: build_doc/Kicad schematic files/aquaponics system.sch (KiCad schematic (older format))
At the start: 18 parts

Commit message: bit more schematic stuff
Parts:
- removed P?: BNC, symbol BNC
- added IC? (x2): DS18B20, 1wire-TO92-, symbol DS18B20
Connections:
- wire segments 49 -> 54
Other:
- note removed: "DS18B20"
- moved on the sheet: R?, SW?

Commit message: started looking at kicad schematic
Parts:
- removed IC? (x2): DS18B20, 1wire-TO92-, symbol DS18B20
Connections:
- wire segments 54 -> 52
Changed lines of the file:
@@
-EESchema Schematic File Version 2
+EESchema Schematic File Version 2  date Thu 07 Apr 2016 10:35:14 BST
 LIBS:power
 LIBS:device
@@
 LIBS:contrib
 LIBS:valves
-LIBS:ESP8266
-LIBS:1wire
 LIBS:aquaponics system-cache
-EELAYER 25 0
+EELAYER 25  0
 EELAYER END
-$Descr A4 11693 8268
+$Descr A4 11700 8267
 encoding utf-8
 Sheet 1 1
 Title "Aquaponics System"
-Date "Fri 26 Jun 2015"
+Date "7 apr 2016"
 Rev "1.0"
 Comp ""
@@
 F 0 "R?" V 7592 3098 50  0000 C CNN
 F 1 "4.7K" V 7416 3104 50  0000 C CNN
-F 2 "" V 7430 3100 30  0000 C CNN
-F 3 "" H 7500 3100 30  0000 C CNN
 	1    7500 3100
 	-1   0    0    -1
@@
 F 0 "SW?" H 1400 5050 50  0000 C CNN
 F 1 "SPST" H 1700 4900 50  0001 C CNN
-F 2 "" H 1700 5000 60  0000 C CNN
-F 3 "" H 1700 5000 60  0000 C CNN
 	1    1700 5000
 	0    1    1    0
@@
 F 0 "SW?" H 2150 5350 50  0000 C CNN
 F 1 "SPST" H 2450 5200 50  0001 C CNN
-F 2 "" H 2450 5300 60  0000 C CNN
-F 3 "" H 2450 5300 60  0000 C CNN
 	1    2450 5300
 	0    1    1    0
@@
 F 1 "SPST" H 2700 5300 50  0001 C CNN
 F 2 "~" H 2700 5400 60  0001 C CNN
-F 3 "" H 2700 5400 60  0000 C CNN
 	1    2700 5400
 	0    1    1    0
@@
 F 0 "R?" V 3630 4200 50  0000 C CNN
 F 1 "1.2K" V 3472 4204 50  0000 C CNN
-F 2 "" V 3480 4200 30  0000 C CNN
-F 3 "" H 3550 4200 30  0000 C CNN
 	1    3550 4200
 	0    1    1    0
@@
 F 0 "R?" V 3630 4450 50  0000 C CNN
 F 1 "1.2K" V 3480 4450 50  0000 C CNN
-F 2 "" V 3480 4450 30  0000 C CNN
-F 3 "" H 3550 4450 30  0000 C CNN
 	1    3550 4450
 	0    1    1    0
@@
 F 0 "R?" V 3630 4700 50  0000 C CNN
 F 1 "1.2K" V 3475 4703 50  0000 C CNN
-F 2 "" V 3480 4700 30  0000 C CNN
-F 3 "" H 3550 4700 30  0000 C CNN
 	1    3550 4700
 	0    1    1    0
@@
 F 0 "#PWR?" H 3550 6200 50  0001 C CNN
 F 1 "GND" H 3550 6300 50  0000 C CNN
-F 2 "" H 3550 6450 60  0000 C CNN
-F 3 "" H 3550 6450 60  0000 C CNN
 	1    3550 6450
 	1    0    0    -1
@@
 F 0 "R?" V 3630 4950 50  0000 C CNN
 F 1 "1.2K" V 3475 4953 50  0000 C CNN
-F 2 "" V 3480 4950 30  0000 C CNN
-F 3 "" H 3550 4950 30  0000 C CNN
 	1    3550 4950
 	0    1    1    0
@@
 F 0 "R?" V 3630 5200 50  0000 C CNN
 F 1 "1.2K" V 3475 5203 50  0000 C CNN
-F 2 "" V 3480 5200 30  0000 C CNN
-F 3 "" H 3550 5200 30  0000 C CNN
 	1    3550 5200
 	0    1    1    0
@@
 F 0 "SW?" H 1650 5150 50  0000 C CNN
 F 1 "SPST" H 1950 5000 50  0001 C CNN
-F 2 "" H 1950 5100 60  0000 C CNN
-F 3 "" H 1950 5100 60  0000 C CNN
 	1    1950 5100
 	0    1    1    0
@@
 F 0 "SW?" H 1900 5250 50  0000 C CNN
 F 1 "SPST" H 2200 5100 50  0001 C CNN
-F 2 "" H 2200 5200 60  0000 C CNN
-F 3 "" H 2200 5200 60  0000 C CNN
 	1    2200 5200
 	0    1    1    0
@@
 F 0 "#PWR?" H 5400 2300 50  0001 C CNN
 F 1 "+3V3" H 5400 2590 50  0000 C CNN
-F 2 "" H 5400 2450 60  0000 C CNN
-F 3 "" H 5400 2450 60  0000 C CNN
 	1    5400 2450
 	1    0    0    -1
@@
 F 0 "C?" H 6225 2900 50  0000 L CNN
 F 1 "100n" H 6225 2700 50  0000 L CNN
-F 2 "" H 6238 2650 30  0000 C CNN
-F 3 "" H 6200 2800 60  0000 C CNN
 	1    6200 2800
 	-1   0    0    1
@@
 F 0 "#PWR?" H 6200 2750 50  0001 C CNN
 F 1 "GND" H 6200 2850 50  0000 C CNN
-F 2 "" H 6200 3000 60  0000 C CNN
-F 3 "" H 6200 3000 60  0000 C CNN
 	1    6200 3000
 	1    0    0    -1
@@
 F 0 "R?" V 6780 4450 50  0000 C CNN
 F 1 "10K" V 6700 4450 50  0000 C CNN
-F 2 "" V 6630 4450 30  0000 C CNN
-F 3 "" H 6700 4450 30  0000 C CNN
 	1    6700 4450
 	1    0    0    -1
@@
 F 0 "R?" V 6780 3100 50  0000 C CNN
 F 1 "10K" V 6700 3100 50  0000 C CNN
-F 2 "" V 6630 3100 30  0000 C CNN
-F 3 "" H 6700 3100 30  0000 C CNN
 	1    6700 3100
 	1    0    0    -1
@@
 F 0 "R?" V 3980 3050 50  0000 C CNN
 F 1 "10K" V 3900 3050 50  0000 C CNN
-F 2 "" V 3830 3050 30  0000 C CNN
-F 3 "" H 3900 3050 30  0000 C CNN
 	1    3900 3050
 	1    0    0    -1
@@
 F 0 "R?" V 3780 3050 50  0000 C CNN
 F 1 "10K" V 3700 3050 50  0000 C CNN
-F 2 "" V 3630 3050 30  0000 C CNN
-F 3 "" H 3700 3050 30  0000 C CNN
 	1    3700 3050
 	1    0    0    -1
@@
 F 0 "U?" H 5400 3600 50  0000 C CNN
 F 1 "ESP-12" H 5400 3800 50  0000 C CNN
-F 2 "" H 5400 3700 50  0001 C CNN
-F 3 "" H 5400 3700 50  0001 C CNN
 	1    5400 3700
 	1    0    0    -1
@@
 Wire Wire Line
 	6200 3000 6200 2950
-$Comp
-L DS18B20 IC?
-U 3 1 55929CD9
-P 7850 3900
-F 0 "IC?" H 8075 3925 50  0000 L BNN
-F 1 "DS18B20" H 8075 3825 50  0000 L BNN
-F 2 "1wire-TO92-" H 7850 4050 50  0001 C CNN
-F 3 "" H 7850 3900 60  0000 C CNN
-	3    7850 3900
-	1    0    0    -1
-$EndComp
-$Comp
-L DS18B20 IC?
-U 2 1 5592A02C
-P 7850 3900
-F 0 "IC?" H 8075 3925 50  0000 L BNN
-F 1 "DS18B20" H 8075 3825 50  0000 L BNN
-F 2 "1wire-TO92-" H 7850 4050 50  0001 C CNN
-F 3 "" H 7850 3900 60  0000 C CNN
-	2    7850 3900
-	1    0    0    -1
-$EndComp
 Wire Wire Line
 	6300 3900 7500 3900
-Wire Wire Line
-	7500 3900 7650 3900
 Connection ~ 7500 3900
-Wire Wire Line
-	7850 2600 7850 3600
 Connection ~ 6700 2600
 Wire Wire Line

Commit message: Finished Schematic & added little bit more comments to waterelf
Parts:
- removed R? (x5): 1.2K, symbol R
- removed SW? (x4): SPST, symbol SPST
- removed SW?: SPST, ~, symbol SPST
- added P? (x3): PUMP, symbol PUMP
- added Q? (x3): SI2302DS, SOT-23, symbol SI2302DS
- added R? (x4): 10K, symbol R
- added U?: DS18B20, symbol DS18B20
- added U?: AM2302, symbol DHT22/AM2302
- added U?: XY-FSK, symbol XY-FSK
- added U?: PH_MODULE, symbol PH_MODULE
- added U?: TSL2591_MODULE, symbol TSL2591_MODULE
- added U?: MCP23008, symbol MCP23008
- added U? (x3): HC-SR04, symbol HC-SR04
- R?: value 4.7K -> 10K
Connections:
- net labels added: +3.3VP
- wire segments 52 -> 163
Other:
- note added: "433MHZ TRANS"
- note added: "ADAFRUIT ESP HUZZAH MODULE"
- note added: "AIR TEMP/HUMID"
- note added: "GROWBED 1"
- note added: "GROWBED 2"
- note added: "GROWBED 3"
- note added: "LUX SENSOR"
- note added: "WATER TEMP PROBE"
- note removed: "TEMP PROBE"
- note removed: "WATER\nLEVEL\nSWITCHES"
- moved on the sheet: C?, R?, U?

Commit message: updated schematic, added decoupling
Parts:
- added C?: 100n, symbol C
Connections:
- wire segments 163 -> 169
Other:
- moved on the sheet: U?
Changed lines of the file:
@@
-EESchema Schematic File Version 2  date Sun 10 Apr 2016 16:23:37 BST
+EESchema Schematic File Version 2  date Tue 12 Apr 2016 09:16:11 BST
 LIBS:power
 LIBS:device
@@
 Sheet 1 1
 Title "Aquaponics System"
-Date "10 apr 2016"
-Rev "1.2"
+Date "12 apr 2016"
+Rev "1.3"
 Comp ""
 Comment1 ""
@@
 $EndDescr
 Wire Wire Line
-	4350 2150 4450 2150
-Wire Wire Line
-	4350 1750 4450 1750
-Wire Wire Line
-	4350 1550 4450 1550
-Wire Wire Line
-	4350 1350 5550 1350
+	1300 1950 1300 2000
+Connection ~ 1300 1500
+Wire Wire Line
+	1300 1450 1300 1500
+Connection ~ 4350 1850
+Connection ~ 4350 1100
+Wire Wire Line
+	4350 1100 4350 1850
+Wire Wire Line
+	4350 1850 4350 2550
+Wire Wire Line
+	4350 2550 3900 2550
+Wire Wire Line
+	4350 1850 4200 1850
+Wire Wire Line
+	2800 1850 2200 1850
+Connection ~ 4450 2400
+Wire Wire Line
+	4450 2400 3500 2400
+Wire Wire Line
+	4450 2150 4200 2150
+Wire Wire Line
+	4450 1750 4200 1750
+Wire Wire Line
+	4200 1550 4450 1550
+Wire Wire Line
+	4200 1350 5550 1350
 Wire Wire Line
 	4900 3050 4900 3700
 Wire Wire Line
-	7600 3450 7600 1100
-Wire Wire Line
-	4350 3400 4350 4000
-Wire Wire Line
-	4350 4000 4350 4500
-Wire Wire Line
-	4350 4500 4350 5600
-Wire Wire Line
-	4350 3400 3650 3400
-Connection ~ 4650 1850
-Wire Wire Line
-	4650 1100 4650 1850
-Wire Wire Line
-	4650 1850 4650 2500
+	7600 1100 7600 3450
+Wire Wire Line
+	4000 3400 4000 4000
+Wire Wire Line
+	4000 4000 4000 4500
+Wire Wire Line
+	4000 4500 4000 5600
+Wire Wire Line
+	4000 3400 3650 3400
 Wire Wire Line
 	5600 1100 5600 1000
@@
 	1900 2100 1300 2100
 Wire Wire Line
-	1900 1500 1000 1500
+	1900 1500 1300 1500
+Wire Wire Line
+	1300 1500 1000 1500
 Connection ~ 1300 2500
 Wire Wire Line
@@
 	2200 5000 2200 3900
 Wire Wire Line
-	4350 5600 3650 5600
-Wire Wire Line
-	3900 5450 3900 4350
-Wire Wire Line
-	3900 4350 3900 3250
-Wire Wire Line
-	3900 3250 3900 2500
-Wire Wire Line
-	2850 1350 2850 1100
-Wire Wire Line
-	4150 3900 4150 4650
-Wire Wire Line
-	4150 3900 5350 3900
-Wire Wire Line
-	4350 4000 5350 4000
+	4000 5600 3650 5600
+Wire Wire Line
+	4200 3900 4200 4650
+Wire Wire Line
+	4200 3900 5350 3900
+Wire Wire Line
+	4000 4000 5350 4000
 Connection ~ 3900 3250
 Wire Wire Line
@@
 	1300 1650 1300 1600
 Wire Wire Line
-	1300 1450 1300 1500
-Wire Wire Line
-	2200 2350 2700 2350
-Wire Wire Line
-	2700 2350 2700 2150
-Wire Wire Line
-	2700 2150 2950 2150
-Wire Wire Line
-	2200 1350 2700 1350
-Wire Wire Line
-	2700 1350 2700 1450
-Wire Wire Line
-	2700 1450 2950 1450
+	2200 2350 2550 2350
+Wire Wire Line
+	2550 2350 2550 2150
+Wire Wire Line
+	2200 1350 2550 1350
+Wire Wire Line
+	2550 1350 2550 1450
 Connection ~ 4450 1750
 Connection ~ 4450 6350
@@
 Connection ~ 8400 1100
 Wire Wire Line
-	8400 1100 8400 3450
+	8400 3450 8400 1100
 Wire Notes Line
 	8200 2600 4650 2600
@@
 Connection ~ 7600 3900
 Wire Wire Line
-	8400 4000 7900 4000
-Wire Wire Line
-	7900 4000 7150 4000
+	7150 4000 7900 4000
+Wire Wire Line
+	7900 4000 8400 4000
 Wire Wire Line
 	8500 5250 9100 5250
@@
 	4900 3700 5350 3700
 Wire Wire Line
-	5200 2750 5200 1100
+	5200 1100 5200 2750
 Connection ~ 5200 1100
 Connection ~ 5600 1100
@@
 	9100 3100 7400 3100
 Connection ~ 7400 3100
-Wire Wire Line
-	2850 1350 2950 1350
 Connection ~ 4900 1100
 Wire Wire Line
@@
 Connection ~ 7300 2300
 Connection ~ 4450 1650
-Connection ~ 4650 1100
-Wire Wire Line
-	2150 1850 2950 1850
 Wire Wire Line
 	1300 1100 1300 1150
-Wire Wire Line
-	1300 2000 1300 1950
 Wire Wire Line
 	1300 2100 1300 2150
@@
 Connection ~ 2200 6350
 Wire Wire Line
-	3650 3250 3900 3250
-Connection ~ 2850 1350
-Wire Wire Line
-	3900 5450 3650 5450
+	3900 3250 3650 3250
+Wire Wire Line
+	3650 5450 3900 5450
 Connection ~ 3900 4350
-Connection ~ 4350 4000
-Wire Wire Line
-	5350 4100 4250 4100
-Wire Wire Line
-	4250 4100 4250 3550
-Wire Wire Line
-	4250 3550 3650 3550
-Wire Wire Line
-	3650 5750 4050 5750
-Wire Wire Line
-	4050 5750 4050 3800
-Wire Wire Line
-	4050 3800 5350 3800
-Wire Wire Line
-	4150 4650 3650 4650
-Wire Wire Line
-	3650 4500 4350 4500
-Connection ~ 4350 4500
+Connection ~ 4000 4000
+Wire Wire Line
+	5350 4100 4300 4100
+Wire Wire Line
+	4300 4100 4300 3550
+Wire Wire Line
+	4300 3550 3650 3550
+Wire Wire Line
+	3650 5750 4100 5750
+Wire Wire Line
+	4100 5750 4100 3800
+Wire Wire Line
+	4100 3800 5350 3800
+Wire Wire Line
+	4200 4650 3650 4650
+Wire Wire Line
+	3650 4500 4000 4500
+Connection ~ 4000 4500
 Wire Wire Line
 	4450 1550 4450 1650
@@
 	4450 1750 4450 2150
 Wire Wire Line
-	4450 2150 4450 3700
+	4450 2150 4450 2400
+Wire Wire Line
+	4450 2400 4450 3700
 Wire Wire Line
 	4450 3700 4450 4800
@@
 Wire Wire Line
 	4450 5900 4450 6350
-Connection ~ 2200 3900
 Wire Wire Line
 	8400 4650 8400 4000
@@
 	1300 2500 1900 2500
 Wire Wire Line
-	1900 2000 1100 2000
+	1900 2000 1300 2000
+Wire Wire Line
+	1300 2000 1100 2000
 Wire Wire Line
 	1100 2000 1100 4100
@@
 	2100 1100 2100 950
 Connection ~ 2100 1100
-Wire Wire Line
-	3900 2500 4650 2500
 Connection ~ 7900 1100
 Connection ~ 7600 1100
@@
 	5200 3500 5200 3050
 Wire Wire Line
+	5650 1450 4200 1450
+Wire Wire Line
+	4450 1650 4200 1650
+Wire Wire Line
+	3500 2700 3900 2700
+Connection ~ 3900 2700
+Wire Wire Line
+	2550 1450 2800 1450
+Wire Wire Line
+	2550 2150 2800 2150
+Wire Wire Line
+	3900 5450 3900 4350
+Wire Wire Line
+	3900 4350 3900 3250
+Wire Wire Line
+	3900 3250 3900 2700
+Wire Wire Line
+	3900 2700 3900 2550
+Wire Wire Line
 	8850 1100 8400 1100
 Wire Wire Line
@@
 	5200 1100 4900 1100
 Wire Wire Line
-	4900 1100 4650 1100
-Wire Wire Line
-	4650 1100 2850 1100
-Wire Wire Line
-	5650 1450 4350 1450
-Wire Wire Line
-	4350 1650 4450 1650
-Wire Wire Line
-	4350 1850 4650 1850
+	4900 1100 4350 1100
+Wire Wire Line
+	4350 1100 2700 1100
+Wire Wire Line
+	2700 1100 2700 1350
+Wire Wire Line
+	2700 1350 2800 1350
+Connection ~ 1300 2000
+$Comp
+L C C?
+U 1 1 570CAB2B
+P 3500 2550
+F 0 "C?" H 3550 2450 50  0000 L CNN
+F 1 "100n" H 3550 2650 50  0000 L CNN
+	1    3500 2550
+	-1   0    0    1
+$EndComp
 $Comp
 L +3.3VP #PWR?
@@
 L MCP23008 U?
 U 1 1 5707C789
-P 3650 1700
-F 0 "U?" H 3650 2150 70  0000 C CNN
-F 1 "MCP23008" H 3650 1100 70  0000 C CNN
-	1    3650 1700
-	-1   0    0    -1
-$EndComp
+P 3500 1700
+F 0 "U?" H 3500 2150 70  0000 C CNN
+F 1 "MCP23008" H 3500 1100 70  0000 C CNN
+	1    3500 1700
+	-1   0    0    -1
+$EndComp

Commit message: updated BOM and schematic
Parts:
- added C?: 10uF, symbol C
- added C?: 100uF, symbol C
- added IC?: LM1117-33, symbol LM1117
- U?: value ESP-12 -> ESP-12F
Connections:
- net labels added: +3.3V, +5V
- net labels removed: +3.3VP
- wire segments 169 -> 121

Commit message: tweaked schematic
Parts:
- C?: value 100n -> 100nF
Changed lines of the file:
@@
-EESchema Schematic File Version 2  date Fri 15 Apr 2016 12:30:55 BST
+EESchema Schematic File Version 2  date Fri 15 Apr 2016 14:33:55 BST
 LIBS:power
 LIBS:device
@@
 P 3500 2550
 F 0 "C?" H 3550 2450 50  0000 L CNN
-F 1 "100n" H 3550 2650 50  0000 L CNN
+F 1 "100nF" H 3550 2650 50  0000 L CNN
 	1    3500 2550
 	-1   0    0    1
