File: build_doc/Kicad_schematic_files/aquaponics-system.sch (KiCad schematic (older format))
At the start: 30 parts

Commit message: squashed libraries, tweaked doc
Parts:
- removed U?: DS18B20, symbol DS18B20
- added U?: MAX31820/DS18B20, symbol MAX31820
Changed lines of the file:
@@
-EESchema Schematic File Version 2  date Fri 15 Apr 2016 14:33:55 BST
+EESchema Schematic File Version 2  date Tue 19 Apr 2016 15:55:54 BST
 LIBS:power
 LIBS:device
@@
 LIBS:contrib
 LIBS:valves
-LIBS:ESP8266
 LIBS:waterelf
-LIBS:aquaponics system-cache
+LIBS:aquaponics-system-cache
 EELAYER 25  0
 EELAYER END
@@
 Sheet 1 1
 Title "Aquaponics System"
-Date "15 apr 2016"
-Rev "1.3"
+Date "19 apr 2016"
+Rev "1.4"
 Comp ""
 Comment1 ""
@@
 Comment4 ""
 $EndDescr
+$Comp
+L MAX31820 U?
+U 1 1 571645C2
+P 9600 4650
+F 0 "U?" H 9450 4900 50  0000 C CNN
+F 1 "MAX31820/DS18B20" H 9750 4400 50  0000 C CNN
+	1    9600 4650
+	1    0    0    -1
+$EndComp
 Connection ~ 2700 1100
 Wire Wire Line
@@
 	1    0    0    -1
 $EndComp
-$Comp
-L DS18B20 U?
-U 1 1 57078EA3
-P 9600 4650
-F 0 "U?" H 9450 4900 50  0000 C CNN
-F 1 "DS18B20" H 9600 4400 50  0000 C CNN
-	1    9600 4650
-	1    0    0    -1
-$EndComp

Commit message: tweaked schematic, updated BOM with uk ebay links
Parts:
- Q? (x3): symbol SI2302DS -> Si2302DS
- U?: symbol PH_MODULE -> pH_MODULE
Changed lines of the file:
@@
-EESchema Schematic File Version 2  date Tue 19 Apr 2016 15:55:54 BST
+EESchema Schematic File Version 2
+LIBS:aquaponics-system-rescue
 LIBS:power
 LIBS:device
@@
 LIBS:waterelf
 LIBS:aquaponics-system-cache
-EELAYER 25  0
+EELAYER 25 0
 EELAYER END
-$Descr A4 11700 8267
+$Descr A4 11693 8268
 encoding utf-8
 Sheet 1 1
@@
 F 0 "U?" H 9450 4900 50  0000 C CNN
 F 1 "MAX31820/DS18B20" H 9750 4400 50  0000 C CNN
+F 2 "" H 9600 4650 60  0001 C CNN
+F 3 "" H 9600 4650 60  0001 C CNN
 	1    9600 4650
 	1    0    0    -1
@@
 F 0 "#PWR?" H 2200 6650 50  0001 C CNN
 F 1 "+3.3V" H 2200 6940 50  0000 C CNN
+F 2 "" H 2200 6800 60  0001 C CNN
+F 3 "" H 2200 6800 60  0001 C CNN
 	1    2200 6800
 	1    0    0    -1
@@
 F 0 "C?" H 2225 7350 50  0000 L CNN
 F 1 "100uF" H 2225 7150 50  0000 L CNN
+F 2 "" H 2200 7250 60  0001 C CNN
+F 3 "" H 2200 7250 60  0001 C CNN
 	1    2200 7250
 	1    0    0    -1
@@
 F 0 "IC?" H 1800 6650 50  0000 L BNN
 F 1 "LM1117-33" H 1800 6550 50  0000 L BNN
+F 2 "" H 1700 6950 60  0001 C CNN
+F 3 "" H 1700 6950 60  0001 C CNN
 	1    1700 6950
 	1    0    0    -1
@@
 F 0 "C?" H 1225 7350 50  0000 L CNN
 F 1 "10uF" H 1225 7150 50  0000 L CNN
+F 2 "" H 1200 7250 60  0001 C CNN
+F 3 "" H 1200 7250 60  0001 C CNN
 	1    1200 7250
 	1    0    0    -1
@@
 F 0 "#PWR?" H 1200 6650 50  0001 C CNN
 F 1 "+5V" H 1200 6940 50  0000 C CNN
+F 2 "" H 1200 6800 60  0001 C CNN
+F 3 "" H 1200 6800 60  0001 C CNN
 	1    1200 6800
 	1    0    0    -1
@@
 F 0 "C?" H 3550 2450 50  0000 L CNN
 F 1 "100nF" H 3550 2650 50  0000 L CNN
+F 2 "" H 3500 2550 60  0001 C CNN
+F 3 "" H 3500 2550 60  0001 C CNN
 	1    3500 2550
 	-1   0    0    1
@@
 F 0 "U?" H 2950 5900 60  0000 C CNN
 F 1 "HC-SR04" H 3100 5150 60  0000 C CNN
+F 2 "" H 3100 5600 60  0001 C CNN
+F 3 "" H 3100 5600 60  0001 C CNN
 	1    3100 5600
 	-1   0    0    -1
@@
 F 0 "U?" H 2950 4800 60  0000 C CNN
 F 1 "HC-SR04" H 3100 4050 60  0000 C CNN
+F 2 "" H 3100 4500 60  0001 C CNN
+F 3 "" H 3100 4500 60  0001 C CNN
 	1    3100 4500
 	-1   0    0    -1
@@
 F 0 "P?" H 1800 5900 60  0000 C CNN
 F 1 "PUMP" H 1800 5400 60  0000 C CNN
+F 2 "" H 1800 5650 60  0001 C CNN
+F 3 "" H 1800 5650 60  0001 C CNN
 	1    1800 5650
 	0    1    1    0
@@
 F 0 "P?" H 1800 4800 60  0000 C CNN
 F 1 "PUMP" H 1800 4300 60  0000 C CNN
+F 2 "" H 1800 4550 60  0001 C CNN
+F 3 "" H 1800 4550 60  0001 C CNN
 	1    1800 4550
 	0    1    1    0
@@
 F 0 "U?" H 2950 3700 60  0000 C CNN
 F 1 "HC-SR04" H 3100 2950 60  0000 C CNN
+F 2 "" H 3100 3400 60  0001 C CNN
+F 3 "" H 3100 3400 60  0001 C CNN
 	1    3100 3400
 	-1   0    0    -1
@@
 F 0 "P?" H 1800 3700 60  0000 C CNN
 F 1 "PUMP" H 1800 3200 60  0000 C CNN
+F 2 "" H 1800 3450 60  0001 C CNN
+F 3 "" H 1800 3450 60  0001 C CNN
 	1    1800 3450
 	0    1    1    0
@@
 F 0 "R?" V 1380 1300 50  0000 C CNN
 F 1 "10K" V 1300 1300 50  0000 C CNN
+F 2 "" H 1300 1300 60  0001 C CNN
+F 3 "" H 1300 1300 60  0001 C CNN
 	1    1300 1300
 	1    0    0    -1
@@
 F 0 "R?" V 1380 1800 50  0000 C CNN
 F 1 "10K" V 1300 1800 50  0000 C CNN
+F 2 "" H 1300 1800 60  0001 C CNN
+F 3 "" H 1300 1800 60  0001 C CNN
 	1    1300 1800
 	1    0    0    -1
@@
 F 0 "R?" V 1380 2300 50  0000 C CNN
 F 1 "10K" V 1300 2300 50  0000 C CNN
+F 2 "" H 1300 2300 60  0001 C CNN
+F 3 "" H 1300 2300 60  0001 C CNN
 	1    1300 2300
 	1    0    0    -1
 $EndComp
 $Comp
-L SI2302DS Q?
+L Si2302DS Q?
 U 1 1 5707CB2F
 P 2000 1800
@@
 F 1 "SI2302DS" H 2200 1800 50  0000 L CNN
 F 2 "SOT-23" H 2200 1700 50  0000 L CIN
+F 3 "" H 2000 1800 60  0001 C CNN
 	1    2000 1800
 	-1   0    0    -1
 $EndComp
 $Comp
-L SI2302DS Q?
+L Si2302DS Q?
 U 1 1 5707CB25
 P 2000 2300
@@
 F 1 "SI2302DS" H 2200 2300 50  0000 L CNN
 F 2 "SOT-23" H 2200 2200 50  0000 L CIN
+F 3 "" H 2000 2300 60  0001 C CNN
 	1    2000 2300
 	-1   0    0    -1
 $EndComp
 $Comp
-L SI2302DS Q?
+L Si2302DS Q?
 U 1 1 5707CB07
 P 2000 1300
@@
 F 1 "SI2302DS" H 2200 1300 50  0000 L CNN
 F 2 "SOT-23" H 2200 1200 50  0000 L CIN
+F 3 "" H 2000 1300 60  0001 C CNN
 	1    2000 1300
 	-1   0    0    -1
@@
 F 0 "U?" H 3500 2150 70  0000 C CNN
 F 1 "MCP23008" H 3500 1100 70  0000 C CNN
+F 2 "" H 3500 1700 60  0001 C CNN
+F 3 "" H 3500 1700 60  0001 C CNN
 	1    3500 1700
 	-1   0    0    -1
@@
 LUX SENSOR
 $Comp
-L PH_MODULE U?
+L pH_MODULE U?
 U 1 1 5707B2A1
 P 9650 2000
 F 0 "U?" H 9500 2300 60  0000 C CNN
 F 1 "PH_MODULE" H 9650 1550 60  0000 C CNN
+F 2 "" H 9650 2000 60  0001 C CNN
+F 3 "" H 9650 2000 60  0001 C CNN
 	1    9650 2000
 	1    0    0    -1
@@
 F 0 "U?" H 9500 3250 60  0000 C CNN
 F 1 "TSL2591_MODULE" H 9750 2500 60  0000 C CNN
+F 2 "" H 9650 2950 60  0001 C CNN
+F 3 "" H 9650 2950 60  0001 C CNN
 	1    9650 2950
 	1    0    0    -1
@@
 F 0 "U?" H 9500 5700 60  0000 C CNN
 F 1 "XY-FSK" H 9550 5100 60  0000 C CNN
+F 2 "" H 9650 5400 60  0001 C CNN
+F 3 "" H 9650 5400 60  0001 C CNN
 	1    9650 5400
 	1    0    0    -1
@@
 F 0 "R?" V 7992 3598 50  0000 C CNN
 F 1 "10K" V 7816 3604 50  0000 C CNN
+F 2 "" H 7900 3600 60  0001 C CNN
+F 3 "" H 7900 3600 60  0001 C CNN
 	1    7900 3600
 	-1   0    0    -1
@@
 F 0 "U?" H 9500 4200 60  0000 C CNN
 F 1 "AM2302" H 9550 3600 60  0000 C CNN
+F 2 "" H 9650 3900 60  0001 C CNN
+F 3 "" H 9650 3900 60  0001 C CNN
 	1    9650 3900
 	1    0    0    -1
@@
 F 0 "R?" V 8492 3598 50  0000 C CNN
 F 1 "10K" V 8316 3604 50  0000 C CNN
+F 2 "" H 8400 3600 60  0001 C CNN
+F 3 "" H 8400 3600 60  0001 C CNN
 	1    8400 3600
 	-1   0    0    -1
@@
 F 0 "#PWR?" H 5600 6200 50  0001 C CNN
 F 1 "GND" H 5600 6300 50  0000 C CNN
+F 2 "" H 5600 6450 60  0001 C CNN
+F 3 "" H 5600 6450 60  0001 C CNN
 	1    5600 6450
 	1    0    0    -1
@@
 F 0 "#PWR?" H 5600 850 50  0001 C CNN
 F 1 "+3V3" H 5600 1140 50  0000 C CNN
+F 2 "" H 5600 1000 60  0001 C CNN
+F 3 "" H 5600 1000 60  0001 C CNN
 	1    5600 1000
 	1    0    0    -1
@@
 F 0 "C?" H 7100 2800 50  0000 L CNN
 F 1 "100n" H 7100 3000 50  0000 L CNN
+F 2 "" H 7050 2900 60  0001 C CNN
+F 3 "" H 7050 2900 60  0001 C CNN
 	1    7050 2900
 	-1   0    0    1
@@
 F 0 "#PWR?" H 7050 2850 50  0001 C CNN
 F 1 "GND" H 7050 2950 50  0000 C CNN
+F 2 "" H 7050 3100 60  0001 C CNN
+F 3 "" H 7050 3100 60  0001 C CNN
 	1    7050 3100
 	1    0    0    -1
@@
 F 0 "R?" V 7500 4500 50  0000 C CNN
 F 1 "10K" V 7700 4500 50  0000 C CNN
+F 2 "" H 7600 4500 60  0001 C CNN
+F 3 "" H 7600 4500 60  0001 C CNN
 	1    7600 4500
 	1    0    0    -1
@@
 F 0 "R?" V 7500 3600 50  0000 C CNN
 F 1 "10K" V 7700 3600 50  0000 C CNN
+F 2 "" H 7600 3600 60  0001 C CNN
+F 3 "" H 7600 3600 60  0001 C CNN
 	1    7600 3600
 	1    0    0    -1
@@
 F 0 "R?" V 5100 2900 50  0000 C CNN
 F 1 "10K" V 5300 2900 50  0000 C CNN
+F 2 "" H 5200 2900 60  0001 C CNN
+F 3 "" H 5200 2900 60  0001 C CNN
 	1    5200 2900
 	1    0    0    -1
@@
 F 0 "R?" V 4800 2900 50  0000 C CNN
 F 1 "10K" V 5000 2900 50  0000 C CNN
+F 2 "" H 4900 2900 60  0001 C CNN
+F 3 "" H 4900 2900 60  0001 C CNN
 	1    4900 2900
 	1    0    0    -1
@@
 F 0 "U?" H 6250 3700 50  0000 C CNN
 F 1 "ESP-12F" H 6250 3900 50  0000 C CNN
+F 2 "" H 6250 3800 60  0001 C CNN
+F 3 "" H 6250 3800 60  0001 C CNN
 	1    6250 3800
 	1    0    0    -1

Commit message: latest addition to schematic
Parts:
- added D? (x3): 1N4001, symbol D
- added R? (x3): 470R, symbol R
- added S? (x3): Solenoid, symbol Solenoid
Connections:
- net +3V3: now also P?.1 (+ve), P?.1 (+ve), P?.1 (+ve), D?.1 (K), D?.1 (K), D?.1 (K), S?.2, S?.2, S?.2; no longer C?.1, Q?.3 (D), Q?.3 (D), Q?.3 (D), R?.1, R?.1, R?.1, U?.1 (VCC), U?.1 (VCC), U?.1 (VCC)
- net +5V: now also C?.1, U?.1 (VCC), U?.1 (VCC), U?.1 (VCC)
- net GND: now also Q?.2 (S), Q?.2 (S), Q?.2 (S), R?.2, R?.2, R?.2; no longer P?.2 (-ve), P?.2 (-ve), P?.2 (-ve)
- net at U?.10 (GP0): now also R?.1; no longer Q?.1 (G)
- net at U?.13 (GP3): now also R?.1; no longer Q?.1 (G)
- net at U?.17 (GP7): now also R?.1; no longer Q?.1 (G)
- new net: Q?.1 (G), R?.1, R?.2 (x3)
- new net: D?.2 (A), P?.2 (-ve), Q?.3 (D), S?.1 (x3)
Other:
- moved on the sheet: C?, P?, R?
